File: VIC1214Reloaded-1.0-001.kicad_pcb (KiCad board)
At the start: 2 copper layers, 65 x 57.3 mm, 26 parts, among them J101 SJ-3568N, U101 MA156-12-2, U102 SP0256-AL2, U103 LM386, X101 CXO_DIP8

Commit message: Add files via upload
Parts:
- removed R105: 33K, Resistor_THT:R_Axial_DIN0207_L6.3mm_D2.5mm_P7.62mm_Horizontal
- removed R106: 10, Resistor_THT:R_Axial_DIN0207_L6.3mm_D2.5mm_P7.62mm_Horizontal
- removed X101: CXO_DIP8, Oscillator:Oscillator_DIP-8
- added C112: 100uF, Capacitor_THT:CP_Radial_D6.3mm_P2.50mm, F.Cu at (115.6, 102.9)
- added Y101: 3.12MHz, Crystal:Crystal_HC49-U_Horizontal_1EP_style2, F.Cu at (97.4, 83.8)
- C102: value 022 -> 22p; footprint Capacitor_THT:C_Disc_D7.0mm_W2.5mm_P5.00mm -> Capacitor_THT:C_Disc_D5.0mm_W2.5mm_P5.00mm
- C103: value 47p -> 22p
- C104: value 10uF -> 022; footprint Capacitor_THT:CP_Radial_D6.3mm_P2.50mm -> Capacitor_THT:C_Disc_D7.0mm_W2.5mm_P5.00mm
- C105: value 022 -> 10uF; footprint Capacitor_THT:C_Disc_D7.0mm_W2.5mm_P5.00mm -> Capacitor_THT:CP_Radial_D6.3mm_P2.50mm
- C106: value 1uF -> 022; footprint Capacitor_THT:CP_Radial_D6.3mm_P2.50mm -> Capacitor_THT:C_Disc_D7.0mm_W2.5mm_P5.00mm
- C107: value 0.1u -> 1uF; footprint Capacitor_THT:C_Disc_D5.0mm_W2.5mm_P5.00mm -> Capacitor_THT:CP_Radial_D6.3mm_P2.50mm
- C108: value 10uF -> 0.1u; footprint Capacitor_THT:CP_Radial_D6.3mm_P2.50mm -> Capacitor_THT:C_Disc_D5.0mm_W2.5mm_P5.00mm
- C109: value 0.1u -> 10uF; footprint Capacitor_THT:C_Disc_D5.0mm_W2.5mm_P5.00mm -> Capacitor_THT:CP_Radial_D6.3mm_P2.50mm
- C111: value 100uF -> 0.1u; footprint Capacitor_THT:CP_Radial_D6.3mm_P2.50mm -> Capacitor_THT:C_Disc_D5.0mm_W2.5mm_P5.00mm
- R102: value 10 -> 33K
- R104: value 10K -> 10
- moved C104 37.2 mm to (94.1, 92.1)
- moved R104 29.7 mm to (94.0, 98.4), turned to 0 degrees
- moved C111 27.5 mm to (94.0, 101.6), turned to 0 degrees
- moved C102 21.1 mm to (94.0, 79.9), turned to 90 degrees
- moved C103 18.6 mm to (94.0, 82.6), turned to -90 degrees
- moved C108 13.3 mm to (128.3, 101.6)
- moved R102 10.2 mm to (111.8, 92.1)
- moved C105 9.25 mm to (104.1, 106.7), turned to 180 degrees
- moved C109 7.73 mm to (115.6, 108.0), turned to -90 degrees
- moved C110 4.00 mm to (100.3, 124.5)
- moved LK101 3.86 mm to (81.9, 124.5)
- moved R101 3.81 mm to (108.0, 113.0)
- moved U103 3.81 mm to (95.2, 113.0)
- moved C107 3.65 mm to (115.6, 118.1)
- moved C106 2.54 mm to (123.2, 101.6)
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Connections:
- C102 pad 2: GNDA -> GND
- C103 pad 2: Net-(C103-Pad2) -> GND
- C104 pad 1: VCC -> Net-(C104-Pad1)
- C105 pad 1: Net-(C105-Pad1) -> VCC
- C106 pad 1: Net-(C105-Pad1) -> Net-(C106-Pad1)
- C106 pad 2: Net-(C106-Pad2) -> GNDA
- C107 pad 1: VCC -> Net-(C106-Pad1)
- C107 pad 2: GNDA -> Net-(C107-Pad2)
- C108 pad 1: Net-(C108-Pad1) -> VCC
- C108 pad 2: Net-(C108-Pad2) -> GNDA
- C109 pad 2: GNDA -> Net-(C109-Pad2)
- C111 pad 2: Net-(C111-Pad2) -> GNDA
- J101 pad 2: Net-(C111-Pad2) -> Net-(C112-Pad2)
- J101 pad 3: Net-(C111-Pad2) -> Net-(C112-Pad2)
- JP101 pad 2: Net-(C105-Pad1) -> Net-(C106-Pad1)
- R102 pad 1: Net-(C103-Pad1) -> Net-(JP101-Pad1)
- R102 pad 2: Net-(R102-Pad2) -> Net-(C104-Pad1)
- R103 pad 1: Net-(JP101-Pad1) -> Net-(C104-Pad1)
- R103 pad 2: Net-(C102-Pad1) -> Net-(C106-Pad1)
- R104 pad 1: Net-(C103-Pad1) -> Net-(C111-Pad1)
- R104 pad 2: GND -> Net-(C112-Pad1)
- U102 pad 27: Net-(R102-Pad2) -> Net-(C103-Pad1)
- U102 pad 28: GND -> Net-(C102-Pad1)
- U103 pad 1: Net-(C108-Pad1) -> Net-(C109-Pad1)
- U103 pad 5: Net-(C111-Pad1) -> Net-(C112-Pad1)
- U103 pad 7: Net-(C109-Pad1) -> Net-(C110-Pad1)
- U103 pad 8: Net-(C108-Pad2) -> Net-(C109-Pad2)
- VR101 pad 3: Net-(C106-Pad2) -> Net-(C107-Pad2)
Routing:
- net Net-(C111-Pad2): track 55.5 -> 0.00 mm
- net Net-(C106-Pad1): track 0.00 -> 45.0 mm
- net Net-(C105-Pad1): track 43.4 -> 0.00 mm
- net Net-(C112-Pad1): track 0.00 -> 39.6 mm
- net Net-(C112-Pad2): track 0.00 -> 27.7 mm
- net Net-(C108-Pad1): track 22.8 -> 0.00 mm
- net PB7: track 32.2 -> 48.3 mm
- net Net-(C108-Pad2): track 14.2 -> 0.00 mm
- net Net-(C104-Pad1): track 0.00 -> 14.0 mm
- net VCC: track 151.8 -> 138.0 mm
- net Net-(C109-Pad2): track 0.00 -> 13.8 mm
- net Net-(C107-Pad2): track 0.00 -> 12.5 mm
- net Net-(C111-Pad1): track 14.0 -> 3.17 mm
- net Net-(C103-Pad1): track 19.6 -> 9.52 mm
- net Net-(R101-Pad1): track 46.6 -> 56.5 mm
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- removed copper zone on F.Cu, net GND
- removed copper zone on F.Cu, net GNDA
- removed copper zone on B.Cu, net VCC
