File: VIC1214Reloaded-1.0-001.kicad_sch (KiCad schematic)
At the start: 26 parts, among them J101 SJ-3568N, U101 MA156-12-2, U102 SP0256-AL2, U103 LM386, X101 CXO_DIP8

Commit message: Add files via upload
Parts:
- removed R102: 10, Resistor_THT:R_Axial_DIN0207_L6.3mm_D2.5mm_P7.62mm_Horizontal, symbol Device:R
- removed R104: 10K, Resistor_THT:R_Axial_DIN0207_L6.3mm_D2.5mm_P7.62mm_Horizontal, symbol Device:R
- removed X101: CXO_DIP8, Oscillator:Oscillator_DIP-8, symbol Oscillator:CXO_DIP8
- added C103: 22pF, Capacitor_THT:C_Disc_D5.0mm_W2.5mm_P5.00mm, symbol Device:C
- added Y101: 3.12MHz, Crystal:Crystal_HC49-U_Horizontal_1EP_style2, symbol Device:Crystal_GND3_Small
- C102: renamed from C103; value 47pF -> 22pF
- renumbered C102 to C104, C104 to C105, C105 to C106, C106 to C107, C107 to C108, C108 to C109, C109 to C110, C110 to C111, C111 to C112, R103 to R102, R105 to R103, R106 to R104
Connections:
- net GND: now also C102.2, C103.2, Y101.3; no longer U102.28 (XTAL2)
- net at U102.27 (XTAL1): now also C103.1, Y101.1
- net at C102.1: now also U102.28 (XTAL2), Y101.2
Other:
- note added: "Original schematic used a 3.12MHz parallel resonant crystal to control the pitch. It's theoretically possible to use a crystal oscillator AC-coupled to XTAL1 and XTAL2 grounded, but no 3.12MHz oscillators are available. Using a colorburst one will change the tone of the speech."
- note removed: "Original schematic used a 3.12MHz parallel resonant crystal to control the pitch. Replaced with similar TTL Oscillator."
- moved on the sheet: C102
